File: Output.kicad_sch (KiCad schematic)
At the start: 0 parts

Commit message: Finish Output Stage & Finish Schematic
Parts:
- added C: 2200u, symbol Device:C_Polarized
- added C25: 10u, symbol Device:C
- added C26, C27, C28, C29, C30, C31, C32: 100n, symbol Device:C
- added R, R45, R47: 10, symbol Device:R
- added R, R46: 10k, symbol Device:R
- added R48, R49, R50, R51, R52, R53, R54, R55, R60, R61, R69, R70: 1, symbol Device:R
- added U10, U11, U12, U13, U14, U20, U21: NE5532, symbol Amplifier_Operational:NE5532
Connections:
- new net: C25.2, R46.1, U10.3 (+), U10.5 (+)
- new net: R47.2, U10.6 (-), U10.7
- new net: R48.2, U12.6 (-), U12.7
- new net: R50.2, U11.1, U11.2 (-)
- new net: C.1, R.2
- new net: R69.2, U21.6 (-), U21.7
- new net: R54.2, U14.6 (-), U14.7
- new net: R52.2, U13.6 (-), U13.7
- new net: R70.2, U21.1, U21.2 (-)
- new net: R60.2, U20.6 (-), U20.7
- new net: R61.2, U20.1, U20.2 (-)
- new net: R55.2, U14.1, U14.2 (-)
- new net: R49.2, U11.6 (-), U11.7
- new net: R53.2, U13.1, U13.2 (-)
- new net: R45.2, U10.1, U10.2 (-)
- new net: R51.2, U12.1, U12.2 (-)
- new net +15V: C26.1, C27.1, C28.1, C29.1, C30.1, C31.1, C32.1, U10.8 (V+), U11.8 (V+), U12.8 (V+), U13.8 (V+), U14.8 (V+), U20.8 (V+), U21.8 (V+)
- new net BUF_IN_RIGHT: R45.1, R47.1, U11.3 (+), U11.5 (+), U12.3 (+), U12.5 (+), U13.3 (+), U13.5 (+), U14.3 (+), U14.5 (+), U20.3 (+), U20.5 (+), U21.3 (+), U21.5 (+)
- new net BUF_OUT_RIGHT: R.1, R48.1, R49.1, R50.1, R51.1, R52.1, R53.1, R54.1, R55.1, R60.1, R61.1, R69.1, R70.1
- new net GND: C26.2, C27.2, C28.2, C29.2, C30.2, C31.2, C32.2, R.1, U10.4 (V-), U11.4 (V-), U12.4 (V-), U13.4 (V-), U14.4 (V-), U20.4 (V-), U21.4 (V-)
- new net HP_OUT_RIGHT: C.2, R.2
- new net VAS_OUT_RIGHT: C25.1
- new net VBIAS_RIGHT: R46.2
Other:
- note added: "Drivers (Right)"
- note added: "Output Protection and Filtering (RIGHT)"
- note added: "Pre-Driver (RIGHT)"

Commit message: Add missing C values
Parts:
- renumbered C to C?, R to R?
Changed lines of the file:
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@@
 		(dnp no)
 		(fields_autoplaced yes)
-		(property "Reference" "R"
+		(property "Reference" "R?"
 			(at 194.31 39.37 90)
 			(effects
@@
 		(instances
 			(project "Amp"
+				(path "/5faae81d-f66a-438b-a97a-07010798add6/09d140a5-be16-4f38-940b-31221fe1edd1"
+					(reference "R?")
+					(unit 1)
+				)
 				(path "/5faae81d-f66a-438b-a97a-07010798add6/2f5c877b-910c-488b-8e5a-727c90fcde6a"
 					(reference "R73")
@@
 		(on_board yes)
 		(dnp no)
-		(property "Reference" "R"
+		(property "Reference" "R?"
 			(at 213.106 49.53 0)
 			(effects
@@
 		(instances
 			(project "Amp"
+				(path "/5faae81d-f66a-438b-a97a-07010798add6/09d140a5-be16-4f38-940b-31221fe1edd1"
+					(reference "R?")
+					(unit 1)
+				)
 				(path "/5faae81d-f66a-438b-a97a-07010798add6/2f5c877b-910c-488b-8e5a-727c90fcde6a"
 					(reference "R74")
@@
 		(dnp no)
 		(fields_autoplaced yes)
-		(property "Reference" "C"
+		(property "Reference" "C?"
 			(at 203.581 38.1 90)
 			(effects
@@
 		(instances
 			(project "Amp"
+				(path "/5faae81d-f66a-438b-a97a-07010798add6/09d140a5-be16-4f38-940b-31221fe1edd1"
+					(reference "C?")
+					(unit 1)
+				)
 				(path "/5faae81d-f66a-438b-a97a-07010798add6/2f5c877b-910c-488b-8e5a-727c90fcde6a"
 					(reference "C42")
@@
 		(dnp no)
 		(fields_autoplaced yes)
-		(property "Reference" "#PWR"
+		(property "Reference" "#PWR?"
 			(at 210.82 59.69 0)
 			(effects
@@
 		(instances
 			(project "Amp"
+				(path "/5faae81d-f66a-438b-a97a-07010798add6/09d140a5-be16-4f38-940b-31221fe1edd1"
+					(reference "#PWR?")
+					(unit 1)
+				)
 				(path "/5faae81d-f66a-438b-a97a-07010798add6/2f5c877b-910c-488b-8e5a-727c90fcde6a"
 					(reference "#PWR057")

Commit message: Add Footprints
Parts:
- C25, C26, C27, C28, C29, C30, C31, C32: footprint (none) -> Capacitor_SMD:C_0805_2012Metric
- C33: renamed from C?; footprint (none) -> Capacitor_SMD:CP_Elec_10x10
- R45, R46, R47, R48, R49, R50, R51, R52, R53, R54, R55, R60, R61, R69, R70: footprint (none) -> Resistor_SMD:R_0805_2012Metric
- R77, R78: renamed from R?; footprint (none) -> Resistor_SMD:R_0805_2012Metric
- U10, U11, U12, U13, U14, U20, U21: footprint (none) -> Package_SO:SOIC-8_3.9x4.9mm_P1.27mm
Changed lines of the file:
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@@
 			)
 		)
-		(property "Footprint" ""
+		(property "Footprint" "Package_SO:SOIC-8_3.9x4.9mm_P1.27mm"
 			(at 80.01 33.02 0)
 			(effects
@@
 			)
 		)
-		(property "Footprint" ""
+		(property "Footprint" "Package_SO:SOIC-8_3.9x4.9mm_P1.27mm"
 			(at 53.34 102.87 0)
 			(effects
@@
 			)
 		)
-		(property "Footprint" ""
+		(property "Footprint" "Package_SO:SOIC-8_3.9x4.9mm_P1.27mm"
 			(at 128.27 102.87 0)
 			(effects
@@
 			)
 		)
-		(property "Footprint" ""
+		(property "Footprint" "Resistor_SMD:R_0805_2012Metric"
 			(at 86.36 125.222 90)
 			(effects
@@
 			)
 		)
-		(property "Footprint" ""
+		(property "Footprint" "Resistor_SMD:R_0805_2012Metric"
 			(at 86.36 102.362 90)
 			(effects
@@
 			)
 		)
-		(property "Footprint" ""
+		(property "Footprint" "Capacitor_SMD:C_0805_2012Metric"
 			(at 116.5352 147.32 0)
 			(effects
@@
 		(dnp no)
 		(fields_autoplaced yes)
-		(property "Reference" "R?"
+		(property "Reference" "R77"
 			(at 194.31 39.37 90)
 			(effects
@@
 			)
 		)
-		(property "Footprint" ""
+		(property "Footprint" "Resistor_SMD:R_0805_2012Metric"
 			(at 194.31 47.498 90)
 			(effects
@@
 			(project "Amp"
 				(path "/5faae81d-f66a-438b-a97a-07010798add6/09d140a5-be16-4f38-940b-31221fe1edd1"
-					(reference "R?")
+					(reference "R77")
 					(unit 1)
 				)
@@
 			)
 		)
-		(property "Footprint" ""
+		(property "Footprint" "Package_SO:SOIC-8_3.9x4.9mm_P1.27mm"
 			(at 222.25 127 0)
 			(effects
@@
 			)
 		)
-		(property "Footprint" ""
+		(property "Footprint" "Resistor_SMD:R_0805_2012Metric"
 			(at 162.56 125.222 90)
 			(effects
@@
 			)
 		)
-		(property "Footprint" ""
+		(property "Footprint" "Resistor_SMD:R_0805_2012Metric"
 			(at 162.56 85.852 90)
 			(effects
@@
 			)
 		)
-		(property "Footprint" ""
+		(property "Footprint" "Capacitor_SMD:C_0805_2012Metric"
 			(at 58.42 29.5148 0)
 			(effects
@@
 		(on_board yes)
 		(dnp no)
-		(property "Reference" "R?"
+		(property "Reference" "R78"
 			(at 213.106 49.53 0)
 			(effects
@@
 			)
 		)
-		(property "Footprint" ""
+		(property "Footprint" "Resistor_SMD:R_0805_2012Metric"
 			(at 212.598 49.53 90)
 			(effects
@@
 			(project "Amp"
 				(path "/5faae81d-f66a-438b-a97a-07010798add6/09d140a5-be16-4f38-940b-31221fe1edd1"
-					(reference "R?")
+					(reference "R78")
 					(unit 1)
 				)
@@
 			)
 		)
-		(property "Footprint" ""
+		(property "Footprint" "Resistor_SMD:R_0805_2012Metric"
 			(at 233.68 141.732 90)
 			(effects
@@
 			)
 		)
-		(property "Footprint" ""
+		(property "Footprint" "Package_SO:SOIC-8_3.9x4.9mm_P1.27mm"
 			(at 222.25 87.63 0)
 			(effects
@@
 			)
 		)
-		(property "Footprint" ""
+		(property "Footprint" "Capacitor_SMD:C_0805_2012Metric"
 			(at 116.5352 107.95 0)
 			(effects
@@
 			)
 		)
-		(property "Footprint" ""
+		(property "Footprint" "Capacitor_SMD:C_0805_2012Metric"
 			(at 41.6052 147.32 0)
 			(effects
@@
 			)
 		)
-		(property "Footprint" ""
+		(property "Footprint" "Package_SO:SOIC-8_3.9x4.9mm_P1.27mm"
 			(at 200.66 102.87 0)
 			(effects
@@
 			)
 		)
-		(property "Footprint" ""
+		(property "Footprint" "Capacitor_SMD:C_0805_2012Metric"
 			(at 41.6052 107.95 0)
 			(effects
@@
 			)
 		)
-		(property "Footprint" ""
+		(property "Footprint" "Capacitor_SMD:C_0805_2012Metric"
 			(at 25.0952 57.15 0)
 			(effects
@@
 			)
 		)
-		(property "Footprint" ""
+		(property "Footprint" "Package_SO:SOIC-8_3.9x4.9mm_P1.27mm"
 			(at 74.93 127 0)
 			(effects
@@
 		(dnp no)
 		(fields_autoplaced yes)
-		(property "Reference" "C?"
+		(property "Reference" "C33"
 			(at 203.581 38.1 90)
 			(effects
@@
 			)
 		)
-		(property "Footprint" ""
+		(property "Footprint" "Capacitor_SMD:CP_Elec_10x10"
 			(at 208.28 44.7548 0)
 			(effects
@@
 			(project "Amp"
 				(path "/5faae81d-f66a-438b-a97a-07010798add6/09d140a5-be16-4f38-940b-31221fe1edd1"
-					(reference "C?")
+					(reference "C33")
 					(unit 1)
 				)
@@
 			)
 		)
-		(property "Footprint" ""
+		(property "Footprint" "Package_SO:SOIC-8_3.9x4.9mm_P1.27mm"
 			(at 222.25 104.14 0)
 			(effects
@@
 			)
 		)
-		(property "Footprint" ""
+		(property "Footprint" "Resistor_SMD:R_0805_2012Metric"
 			(at 162.56 141.732 90)
 			(effects
@@
 			)
 		)
-		(property "Footprint" ""
+		(property "Footprint" "Package_SO:SOIC-8_3.9x4.9mm_P1.27mm"
 			(at 151.13 127 0)
 			(effects
@@
 			)
 		)
-		(property "Footprint" ""
+		(property "Footprint" "Resistor_SMD:R_0805_2012Metric"
 			(at 86.36 85.852 90)
 			(effects
@@
 			)
 		)
-		(property "Footprint" ""
+		(property "Footprint" "Package_SO:SOIC-8_3.9x4.9mm_P1.27mm"
 			(at 74.93 87.63 0)
 			(effects
@@
 			)
 		)
-		(property "Footprint" ""
+		(property "Footprint" "Resistor_SMD:R_0805_2012Metric"
 			(at 162.56 102.362 90)
 			(effects
@@
 			)
 		)
-		(property "Footprint" ""
+		(property "Footprint" "Resistor_SMD:R_0805_2012Metric"
 			(at 67.818 26.67 90)
 			(effects
@@
 			)
 		)
-		(property "Footprint" ""
+		(property "Footprint" "Package_SO:SOIC-8_3.9x4.9mm_P1.27mm"
 			(at 151.13 104.14 0)
 			(effects
@@
 			)
 		)
-		(property "Footprint" ""
+		(property "Footprint" "Package_SO:SOIC-8_3.9x4.9mm_P1.27mm"
 			(at 128.27 142.24 0)
 			(effects
@@
 			)
 		)
-		(property "Footprint" ""
+		(property "Footprint" "Package_SO:SOIC-8_3.9x4.9mm_P1.27mm"
 			(at 222.25 143.51 0)
 			(effects
@@
 			)
 		)
-		(property "Footprint" ""
+		(property "Footprint" "Package_SO:SOIC-8_3.9x4.9mm_P1.27mm"
 			(at 80.01 52.07 0)
 			(effects
@@
 			)
 		)
-		(property "Footprint" ""
+		(property "Footprint" "Package_SO:SOIC-8_3.9x4.9mm_P1.27mm"
 			(at 53.34 142.24 0)
 			(effects
@@
 			)
 		)
-		(property "Footprint" ""
+		(property "Footprint" "Resistor_SMD:R_0805_2012Metric"
 			(at 86.36 141.732 90)
 			(effects
@@
 			)
 		)
-		(property "Footprint" ""
+		(property "Footprint" "Resistor_SMD:R_0805_2012Metric"
 			(at 233.68 102.362 90)
 			(effects
@@
 		(dnp no)
 		(fields_autoplaced yes)
-		(property "Reference" "#PWR?"
+		(property "Reference" "#PWR0101"
 			(at 210.82 59.69 0)
 			(effects
@@
 			(project "Amp"
 				(path "/5faae81d-f66a-438b-a97a-07010798add6/09d140a5-be16-4f38-940b-31221fe1edd1"
-					(reference "#PWR?")
+					(reference "#PWR0101")
 					(unit 1)
 				)
@@
 			)
 		)
-		(property "Footprint" ""
+		(property "Footprint" "Package_SO:SOIC-8_3.9x4.9mm_P1.27mm"
 			(at 151.13 143.51 0)
 			(effects
@@
 			)
 		)
-		(property "Footprint" ""
+		(property "Footprint" "Package_SO:SOIC-8_3.9x4.9mm_P1.27mm"
 			(at 200.66 142.24 0)
 			(effects
@@
 			)
 		)
-		(property "Footprint" ""
+		(property "Footprint" "Package_SO:SOIC-8_3.9x4.9mm_P1.27mm"
 			(at 74.93 143.51 0)
 			(effects
@@
 			)
 		)
-		(property "Footprint" ""
+		(property "Footprint" "Package_SO:SOIC-8_3.9x4.9mm_P1.27mm"
 			(at 36.83 52.07 0)
 			(effects
@@
 			)
 		)
-		(property "Footprint" ""
+		(property "Footprint" "Package_SO:SOIC-8_3.9x4.9mm_P1.27mm"
 			(at 74.93 104.14 0)
 			(effects
@@
 			)
 		)
-		(property "Footprint" ""
+		(property "Footprint" "Resistor_SMD:R_0805_2012Metric"
 			(at 233.68 85.852 90)
 			(effects
@@
 			)
 		)
-		(property "Footprint" ""
+		(property "Footprint" "Capacitor_SMD:C_0805_2012Metric"
 			(at 188.9252 147.32 0)
 			(effects
@@
 			)
 		)
-		(property "Footprint" ""
+		(property "Footprint" "Resistor_SMD:R_0805_2012Metric"
 			(at 93.98 31.242 90)
 			(effects
@@
 			)
 		)
-		(property "Footprint" ""
+		(property "Footprint" "Package_SO:SOIC-8_3.9x4.9mm_P1.27mm"
 			(at 151.13 87.63 0)
 			(effects
@@
 			)
 		)
-		(property "Footprint" ""
+		(property "Footprint" "Resistor_SMD:R_0805_2012Metric"
 			(at 233.68 125.222 90)
 			(effects
@@
 			)
 		)
-		(property "Footprint" ""
+		(property "Footprint" "Resistor_SMD:R_0805_2012Metric"
 			(at 93.98 50.292 90)
 			(effects
@@
 			)
 		)
-		(property "Footprint" ""
+		(property "Footprint" "Capacitor_SMD:C_0805_2012Metric"
 			(at 188.9252 107.95 0)
 			(effects

Commit message: Add inputs audio and power and correct errors
Parts:
- added C52, C54, C55, C56, C57, C58, C59: 100n, Capacitor_SMD:C_0805_2012Metric, symbol Device:C
- added C53: 10u, Capacitor_SMD:C_0805_2012Metric, symbol Device:C
- added C60: 2200u, Capacitor_SMD:CP_Elec_10x10, symbol Device:C_Polarized
- added J5: AudioJack3, Connector_Audio:Jack_3.5mm_CUI_SJ1-3523N_Horizontal, symbol Connector_Audio:AudioJack3
- added R100, R101, R102, R103, R104, R105, R106, R107, R108, R109, R110, R99: 1, Resistor_SMD:R_0805_2012Metric, symbol Device:R
- added R111, R97, R98: 10, Resistor_SMD:R_0805_2012Metric, symbol Device:R
- added R112, R96: 10k, Resistor_SMD:R_0805_2012Metric, symbol Device:R
- added U31, U32, U33, U34, U35, U36, U37: NE5532, Package_SO:SOIC-8_3.9x4.9mm_P1.27mm, symbol Amplifier_Operational:NE5532
- renumbered C26 to C34, C27 to C35, C28 to C36, C25 to C37, C29 to C38, C30 to C39, C31 to C40, C32 to C41, C33 to C42, R52 to R56, R53 to R57, R54 to R58, R55 to R59, R46 to R62, R49 to R63, R50 to R64, R48 to R65, R51 to R66, R47 to R67, R45 to R68, R60 to R71, R61 to R72, R77 to R73, R78 to R74, R69 to R75, R70 to R76, U13 to U15, U14 to U16, U10 to U17, U11 to U18, U12 to U19, U20 to U22, U21 to U23
Connections:
- net +15V: now also C52.1, C54.1, C55.1, C56.1, C57.1, C58.1, C59.1, U31.8 (V+), U32.8 (V+), U33.8 (V+), U34.8 (V+), U35.8 (V+), U36.8 (V+), U37.8 (V+)
- net GND: now also C52.2, C54.2, C55.2, C56.2, C57.2, C58.2, C59.2, J5.S, R112.1, U31.4 (V-), U32.4 (V-), U33.4 (V-), U34.4 (V-), U35.4 (V-), U36.4 (V-), U37.4 (V-)
- net HP_OUT_RIGHT: now also J5.R
- new net: C60.1, R111.2
- new net: R99.2, U32.6 (-), U32.7
- new net: R108.2, U36.1, U36.2 (-)
- new net: R103.2, U34.6 (-), U34.7
- new net: R104.2, U34.1, U34.2 (-)
- new net: R105.2, U35.6 (-), U35.7
- new net: R101.2, U33.6 (-), U33.7
- new net: R98.2, U31.1, U31.2 (-)
- new net: C53.2, R96.1, U31.3 (+), U31.5 (+)
- new net: R109.2, U37.6 (-), U37.7
- new net: R110.2, U37.1, U37.2 (-)
- new net: R106.2, U35.1, U35.2 (-)
- new net: R97.2, U31.6 (-), U31.7
- new net: R100.2, U32.1, U32.2 (-)
- new net: R107.2, U36.6 (-), U36.7
- new net: R102.2, U33.1, U33.2 (-)
- new net BUF_IN_LEFT: R97.1, R98.1, U32.3 (+), U32.5 (+), U33.3 (+), U33.5 (+), U34.3 (+), U34.5 (+), U35.3 (+), U35.5 (+), U36.3 (+), U36.5 (+), U37.3 (+), U37.5 (+)
- new net BUF_OUT_LEFT: R100.1, R101.1, R102.1, R103.1, R104.1, R105.1, R106.1, R107.1, R108.1, R109.1, R110.1, R111.1, R99.1
- new net HP_OUT_LEFT: C60.2, J5.T, R112.2
- new net VAS_OUT_LEFT: C53.1
- new net VBIAS_LEFT: R96.2
Other:
- note added: "Drivers (LEFT)"
- note added: "Output Protection and Filtering (LEFT)"
- note added: "Pre-Driver (LEFT)"
- moved on the sheet: C34, C35, C36, C37, C38, C39, C40, C41, C42, R56, R57, R58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
